Commit message: car_model colcon

File: src/planning/urdf/main_car/car.xacro (robot description, xacro)
@@ -1,107 +1,10 @@
 <?xml version="1.0"?>
-<robot name="photo_main_car" xmlns:xacro="http://www.ros.org/wiki/xacro">
-  <!-- Approximate dimensions inferred from the reference photo. Units: meters, kg. -->
-  <xacro:property name="base_length" value="0.56"/>
-  <xacro:property name="base_width" value="0.36"/>
-  <xacro:property name="base_height" value="0.08"/>
-  <xacro:property name="ground_clearance" value="0.06"/>
-  <xacro:property name="wheel_radius" value="0.075"/>
-  <xacro:property name="wheel_width" value="0.055"/>
-  <xacro:property name="wheel_x" value="0.205"/>
-  <xacro:property name="wheel_y" value="0.205"/>
-  <xacro:property name="wheel_z" value="${wheel_radius}"/>
-  <xacro:property name="plate_length" value="0.46"/>
-  <xacro:property name="plate_width" value="0.31"/>
-  <xacro:property name="plate_thickness" value="0.012"/>
-  <xacro:property name="plate_z" value="0.21"/>
-  <xacro:property name="top_plate_length" value="0.34"/>
-  <xacro:property name="top_plate_width" value="0.26"/>
-  <xacro:property name="top_plate_thickness" value="0.01"/>
-  <xacro:property name="top_plate_z" value="0.32"/>
-  <xacro:property name="lidar_radius" value="0.105"/>
-  <xacro:property name="lidar_height" value="0.08"/>
-  <xacro:property name="lidar_z" value="0.385"/>
-  <xacro:property name="camera_length" value="0.44"/>
-  <xacro:property name="camera_width" value="0.065"/>
-  <xacro:property name="camera_height" value="0.075"/>
-  <xacro:property name="screen_length" value="0.22"/>
-  <xacro:property name="screen_width" value="0.14"/>
-  <xacro:property name="screen_height" value="0.018"/>
-  <xacro:include filename="car_base.xacro"/>
-  <xacro:include filename="car_wheels.xacro"/>
-  <xacro:include filename="car_radar.xacro"/>
-  <xacro:include filename="car_camera.xacro"/>
-  <material name="mat_black">
-    <color rgba="0.02 0.025 0.03 1.0"/>
-  </material>
-  <material name="mat_dark_grey">
-    <color rgba="0.16 0.17 0.16 1.0"/>
-  </material>
-  <material name="mat_grey">
-    <color rgba="0.45 0.46 0.43 1.0"/>
-  </material>
-  <material name="mat_aluminium">
-    <color rgba="0.78 0.77 0.70 1.0"/>
-  </material>
-  <material name="mat_blue">
-    <color rgba="0.00 0.42 0.85 1.0"/>
-  </material>
-  <material name="mat_glass">
-    <color rgba="0.45 0.82 0.95 0.45"/>
-  </material>
-  <material name="mat_green">
-    <color rgba="0.02 0.42 0.18 1.0"/>
-  </material>
-  <material name="mat_red">
-    <color rgba="0.78 0.08 0.18 1.0"/>
-  </material>
-  <material name="mat_gold">
-    <color rgba="0.90 0.62 0.16 1.0"/>
-  </material>
-  <link name="base_footprint"/>
-  <xacro:photo_car_base
-    base_length="${base_length}"
-    base_width="${base_width}"
-    base_height="${base_height}"
-    ground_clearance="${ground_clearance}"
-    plate_length="${plate_length}"
-    plate_width="${plate_width}"
-    plate_thickness="${plate_thickness}"
-    plate_z="${plate_z}"
-    top_plate_length="${top_plate_length}"
-    top_plate_width="${top_plate_width}"
-    top_plate_thickness="${top_plate_thickness}"
-    top_plate_z="${top_plate_z}"/>
-  <joint name="base_footprint_to_base_link" type="fixed">
-    <parent link="base_footprint"/>
-    <child link="base_link"/>
-    <origin xyz="0 0 ${ground_clearance + base_height / 2.0}" rpy="0 0 0"/>
-  </joint>
-  <xacro:photo_wheel name="front_left" parent="base_link" x="${wheel_x}" y="${wheel_y}" z="${wheel_z - (ground_clearance + base_height / 2.0)}" radius="${wheel_radius}" width="${wheel_width}"/>
-  <xacro:photo_wheel name="front_right" parent="base_link" x="${wheel_x}" y="${-wheel_y}" z="${wheel_z - (ground_clearance + base_height / 2.0)}" radius="${wheel_radius}" width="${wheel_width}"/>
-  <xacro:photo_wheel name="rear_left" parent="base_link" x="${-wheel_x}" y="${wheel_y}" z="${wheel_z - (ground_clearance + base_height / 2.0)}" radius="${wheel_radius}" width="${wheel_width}"/>
-  <xacro:photo_wheel name="rear_right" parent="base_link" x="${-wheel_x}" y="${-wheel_y}" z="${wheel_z - (ground_clearance + base_height / 2.0)}" radius="${wheel_radius}" width="${wheel_width}"/>
-  <xacro:photo_radar
-    parent="base_link"
-    x="0.02"
-    y="0.0"
-    z="${lidar_z - (ground_clearance + base_height / 2.0)}"
-    radius="${lidar_radius}"
-    height="${lidar_height}"/>
-  <xacro:photo_front_camera
-    parent="base_link"
-    x="${base_length / 2.0 + camera_width / 2.0 - 0.015}"
-    y="0.0"
-    z="0.055"
-    length="${camera_length}"
-    width="${camera_width}"
-    height="${camera_height}"/>
-  <xacro:photo_screen
-    parent="base_link"
-    x="-0.08"
-    y="0.045"
-    z="${top_plate_z + 0.03 - (ground_clearance + base_height / 2.0)}"
-    length="${screen_length}"
-    width="${screen_width}"
-    height="${screen_height}"/>
+<robot name="main_car" xmlns:xacro="http://www.ros.org/wiki/xacro">
+  <!-- ==================== 常量 ==================== -->
+  <xacro:property name="PI" value="3.141592653"/>
+  <!-- ==================== 子文件 ==================== -->
+  <xacro:include filename="car_base.xacro"/>     <!-- 底盘 + 车轮 -->
+  <xacro:include filename="car_camera.xacro"/>    <!-- 摄像头 -->
+  <xacro:include filename="car_radar.xacro"/>     <!-- 激光雷达 -->
+  <xacro:include filename="car_gazebo.xacro"/>    <!-- Gazebo 仿真插件 -->
 </robot>

File: src/planning/urdf/main_car/car_base.xacro (robot description, xacro)
@@ -1,183 +1,39 @@
-<?xml version="1.0"?>
+<!-- 底盘 -->
 <robot xmlns:xacro="http://www.ros.org/wiki/xacro">
-  <xacro:macro name="box_inertial" params="mass x y z">
-    <inertial>
-      <mass value="${mass}"/>
-      <origin xyz="0 0 0" rpy="0 0 0"/>
-      <inertia
-        ixx="${mass * (y * y + z * z) / 12.0}"
-        ixy="0"
-        ixz="0"
-        iyy="${mass * (x * x + z * z) / 12.0}"
-        iyz="0"
-        izz="${mass * (x * x + y * y) / 12.0}"/>
-    </inertial>
-  </xacro:macro>
-  <xacro:macro name="cylinder_inertial_z" params="mass radius length">
-    <inertial>
-      <mass value="${mass}"/>
-      <origin xyz="0 0 0" rpy="0 0 0"/>
-      <inertia
-        ixx="${mass * (3.0 * radius * radius + length * length) / 12.0}"
-        ixy="0"
-        ixz="0"
-        iyy="${mass * (3.0 * radius * radius + length * length) / 12.0}"
-        iyz="0"
-        izz="${mass * radius * radius / 2.0}"/>
-    </inertial>
-  </xacro:macro>
-  <xacro:macro name="photo_standoff" params="name parent x y z height radius">
-    <link name="${name}_link">
-      <visual>
-        <origin xyz="0 0 0" rpy="0 0 0"/>
-        <geometry>
-          <cylinder radius="${radius}" length="${height}"/>
-        </geometry>
-        <material name="mat_aluminium"/>
-      </visual>
-      <collision>
-        <origin xyz="0 0 0" rpy="0 0 0"/>
-        <geometry>
-          <cylinder radius="${radius}" length="${height}"/>
-        </geometry>
-      </collision>
-      <xacro:cylinder_inertial_z mass="0.03" radius="${radius}" length="${height}"/>
+    <!-- 车体尺寸 -->
+    <xacro:property name="car_length" value="3.0"/>
+    <xacro:property name="car_width" value="1.5"/>
+    <xacro:property name="car_height" value="0.6"/>
+    <!-- 离地间隙 -->
+    <xacro:property name="ground_height" value="0.2"/>
+    <!-- 包含子文件, 要在参数定义之后, 子文件才能使用父文件的参数 -->
+    <xacro:include filename="car_wheels.xacro"/>
+    <!-- 颜色 -->
+    <material name="yellow">
+        <color rgba="0.9 0.6 0.0 0.7"/>
+    </material>
+    <!-- 根坐标 -->
+    <link name="map"/>
+    <!-- 底盘在map的投影点 -->
+    <link name="base_footprint"/>
+    <!-- 底盘 -->
+    <link name="base_link">
+        <visual>
+            <geometry>
+                <box size="${car_length} ${car_width} ${car_height}"/>
+            </geometry>
+            <material name="yellow"/>
+        </visual>
     </link>
-    <joint name="${name}_joint" type="fixed">
-      <parent link="${parent}"/>
-      <child link="${name}_link"/>
-      <origin xyz="${x} ${y} ${z}" rpy="0 0 0"/>
+    <!-- 投影点关联到地图 -->
+    <joint name="footprint_to_map" type="fixed">
+        <parent link="map"/>
+        <child link="base_footprint"/>
     </joint>
-  </xacro:macro>
-  <xacro:macro name="photo_car_base" params="base_length base_width base_height ground_clearance plate_length plate_width plate_thickness plate_z top_plate_length top_plate_width top_plate_thickness top_plate_z">
-    <link name="base_link">
-      <visual>
-        <origin xyz="0 0 0" rpy="0 0 0"/>
-        <geometry>
-          <box size="${base_length} ${base_width} ${base_height}"/>
-        </geometry>
-        <material name="mat_black"/>
-      </visual>
-      <collision>
-        <origin xyz="0 0 0" rpy="0 0 0"/>
-        <geometry>
-          <box size="${base_length} ${base_width} ${base_height}"/>
-        </geometry>
-      </collision>
-      <xacro:box_inertial mass="2.6" x="${base_length}" y="${base_width}" z="${base_height}"/>
-    </link>
-    <link name="middle_plate_link">
-      <visual>
-        <origin xyz="0 0 0" rpy="0 0 0"/>
-        <geometry>
-          <box size="${plate_length} ${plate_width} ${plate_thickness}"/>
-        </geometry>
-        <material name="mat_aluminium"/>
-      </visual>
-      <collision>
-        <origin xyz="0 0 0" rpy="0 0 0"/>
-        <geometry>
-          <box size="${plate_length} ${plate_width} ${plate_thickness}"/>
-        </geometry>
-      </collision>
-      <xacro:box_inertial mass="0.35" x="${plate_length}" y="${plate_width}" z="${plate_thickness}"/>
-    </link>
-    <joint name="middle_plate_joint" type="fixed">
-      <parent link="base_link"/>
-      <child link="middle_plate_link"/>
-      <origin xyz="0 0 ${plate_z - (ground_clearance + base_height / 2.0)}" rpy="0 0 0"/>
+    <!-- 底盘关联到投影点 -->
+    <joint name="base_to_footprint" type="fixed">
+        <parent link="base_footprint"/>
+        <child link="base_link"/>
+        <origin xyz="0.0 0.0 ${car_height / 2.0 + ground_height}"/>
     </joint>
-    <link name="top_plate_link">
-      <visual>
-        <origin xyz="0 0 0" rpy="0 0 0"/>
-        <geometry>
-          <box size="${top_plate_length} ${top_plate_width} ${top_plate_thickness}"/>
-        </geometry>
-        <material name="mat_aluminium"/>
-      </visual>
-      <collision>
-        <origin xyz="0 0 0" rpy="0 0 0"/>
-        <geometry>
-          <box size="${top_plate_length} ${top_plate_width} ${top_plate_thickness}"/>
-        </geometry>
-      </collision>
-      <xacro:box_inertial mass="0.25" x="${top_plate_length}" y="${top_plate_width}" z="${top_plate_thickness}"/>
-    </link>
-    <joint name="top_plate_joint" type="fixed">
-      <parent link="base_link"/>
-      <child link="top_plate_link"/>
-      <origin xyz="-0.04 0 ${top_plate_z - (ground_clearance + base_height / 2.0)}" rpy="0 0 0"/>
-    </joint>
-    <link name="front_sensor_bar_link">
-      <visual>
-        <origin xyz="0 0 0" rpy="0 0 0"/>
-        <geometry>
-          <box size="0.08 ${base_width + 0.035} 0.095"/>
-        </geometry>
-        <material name="mat_dark_grey"/>
-      </visual>
-      <collision>
-        <origin xyz="0 0 0" rpy="0 0 0"/>
-        <geometry>
-          <box size="0.08 ${base_width + 0.035} 0.095"/>
-        </geometry>
-      </collision>
-      <xacro:box_inertial mass="0.45" x="0.08" y="${base_width + 0.035}" z="0.095"/>
-    </link>
-    <joint name="front_sensor_bar_joint" type="fixed">
-      <parent link="base_link"/>
-      <child link="front_sensor_bar_link"/>
-      <origin xyz="${base_length / 2.0 - 0.018} 0 0.035" rpy="0 0 0"/>
-    </joint>
-    <link name="controller_board_link">
-      <visual>
-        <origin xyz="0 0 0" rpy="0 0 0"/>
-        <geometry>
-          <box size="0.19 0.115 0.016"/>
-        </geometry>
-        <material name="mat_green"/>
-      </visual>
-      <collision>
-        <origin xyz="0 0 0" rpy="0 0 0"/>
-        <geometry>
-          <box size="0.19 0.115 0.016"/>
-        </geometry>
-      </collision>
-      <xacro:box_inertial mass="0.10" x="0.19" y="0.115" z="0.016"/>
-    </link>
-    <joint name="controller_board_joint" type="fixed">
-      <parent link="base_link"/>
-      <child link="controller_board_link"/>
-      <origin xyz="-0.07 -0.16 0.105" rpy="0 0 0"/>
-    </joint>
-    <link name="front_battery_link">
-      <visual>
-        <origin xyz="0 0 0" rpy="0 0 0"/>
-        <geometry>
-          <box size="0.13 0.10 0.07"/>
-        </geometry>
-        <material name="mat_red"/>
-      </visual>
-      <collision>
-        <origin xyz="0 0 0" rpy="0 0 0"/>
-        <geometry>
-          <box size="0.13 0.10 0.07"/>
-        </geometry>
-      </collision>
-      <xacro:box_inertial mass="0.45" x="0.13" y="0.10" z="0.07"/>
-    </link>
-    <joint name="front_battery_joint" type="fixed">
-      <parent link="base_link"/>
-      <child link="front_battery_link"/>
-      <origin xyz="0.235 0.055 -0.01" rpy="0 0 0"/>
-    </joint>
-    <xacro:photo_standoff name="front_left_standoff" parent="base_link" x="0.17" y="0.13" z="0.105" height="0.20" radius="0.008"/>
-    <xacro:photo_standoff name="front_right_standoff" parent="base_link" x="0.17" y="-0.13" z="0.105" height="0.20" radius="0.008"/>
-    <xacro:photo_standoff name="rear_left_standoff" parent="base_link" x="-0.18" y="0.13" z="0.105" height="0.20" radius="0.008"/>
-    <xacro:photo_standoff name="rear_right_standoff" parent="base_link" x="-0.18" y="-0.13" z="0.105" height="0.20" radius="0.008"/>
-    <xacro:photo_standoff name="front_left_top_standoff" parent="base_link" x="0.10" y="0.105" z="0.245" height="0.14" radius="0.006"/>
-    <xacro:photo_standoff name="front_right_top_standoff" parent="base_link" x="0.10" y="-0.105" z="0.245" height="0.14" radius="0.006"/>
-    <xacro:photo_standoff name="rear_left_top_standoff" parent="base_link" x="-0.18" y="0.105" z="0.245" height="0.14" radius="0.006"/>
-    <xacro:photo_standoff name="rear_right_top_standoff" parent="base_link" x="-0.18" y="-0.105" z="0.245" height="0.14" radius="0.006"/>
-  </xacro:macro>
 </robot>

File: src/planning/urdf/main_car/car_camera.xacro (robot description, xacro)
@@ -1,77 +1,30 @@
-<?xml version="1.0"?>
+<!-- 摄像头 -->
 <robot xmlns:xacro="http://www.ros.org/wiki/xacro">
-  <xacro:macro name="photo_front_camera" params="parent x y z length width height">
-    <link name="front_camera_link">
-      <visual>
-        <origin xyz="0 0 0" rpy="0 0 0"/>
-        <geometry>
-          <box size="${width} ${length} ${height}"/>
-        </geometry>
-        <material name="mat_dark_grey"/>
-      </visual>
-      <visual>
-        <origin xyz="${width / 2.0 + 0.003} ${length * 0.28} 0.005" rpy="0 ${pi / 2.0} 0"/>
-        <geometry>
-          <cylinder radius="0.023" length="0.01"/>
-        </geometry>
-        <material name="mat_glass"/>
-      </visual>
-      <visual>
-        <origin xyz="${width / 2.0 + 0.003} 0 0.005" rpy="0 ${pi / 2.0} 0"/>
-        <geometry>
-          <cylinder radius="0.023" length="0.01"/>
-        </geometry>
-        <material name="mat_glass"/>
-      </visual>
-      <visual>
-        <origin xyz="${width / 2.0 + 0.003} ${-length * 0.28} 0.005" rpy="0 ${pi / 2.0} 0"/>
-        <geometry>
-          <cylinder radius="0.023" length="0.01"/>
-        </geometry>
-        <material name="mat_glass"/>
-      </visual>
-      <collision>
-        <origin xyz="0 0 0" rpy="0 0 0"/>
-        <geometry>
-          <box size="${width} ${length} ${height}"/>
-        </geometry>
-      </collision>
-      <xacro:box_inertial mass="0.38" x="${width}" y="${length}" z="${height}"/>
+    <!-- 摄像头尺寸 -->
+    <xacro:property name="camera_length" value="0.1"/>
+    <xacro:property name="camera_width" value="0.8"/>
+    <xacro:property name="camera_height" value="0.2"/>
+    <!-- 摄像头偏移量 -->
+    <xacro:property name="camera_joint_x" value="${car_length / 2.0 - 0.02}"/>
+    <xacro:property name="camera_joint_y" value="0.0"/>
+    <xacro:property name="camera_joint_z" value="${car_height / 2.0 + camera_height / 2.0}"/>
+    <!-- 颜色 -->
+    <material name="red">
+        <color rgba="1.0 0.0 0.0 0.8"/>
+    </material>
+    <!-- 摄像头几何 -->
+    <link name="camera">
+        <visual>
+            <geometry>
+                <box size="${camera_length} ${camera_width} ${camera_height}"/>
+            </geometry>
+            <material name="red"/>
+        </visual>
     </link>
-    <joint name="front_camera_joint" type="fixed">
-      <parent link="${parent}"/>
-      <child link="front_camera_link"/>
-      <origin xyz="${x} ${y} ${z}" rpy="0 0 0"/>
+    <!-- 摄像头关联到base_link -->
+    <joint name="camera2base_link" type="fixed">
+        <parent link="base_link"/>
+        <child link="camera"/>
+        <origin xyz="${camera_joint_x} ${camera_joint_y} ${camera_joint_z}"/>
     </joint>
-  </xacro:macro>
-  <xacro:macro name="photo_screen" params="parent x y z length width height">
-    <link name="top_screen_link">
-      <visual>
-        <origin xyz="0 0 0" rpy="0 0 0"/>
-        <geometry>
-          <box size="${length} ${width} ${height}"/>
-        </geometry>
-        <material name="mat_black"/>
-      </visual>
-      <visual>
-        <origin xyz="0 0 ${height / 2.0 + 0.002}" rpy="0 0 0"/>
-        <geometry>
-          <box size="${length * 0.92} ${width * 0.82} 0.003"/>
-        </geometry>
-        <material name="mat_glass"/>
-      </visual>
-      <collision>
-        <origin xyz="0 0 0" rpy="0 0 0"/>
-        <geometry>
-          <box size="${length} ${width} ${height}"/>
-        </geometry>
-      </collision>
-      <xacro:box_inertial mass="0.12" x="${length}" y="${width}" z="${height}"/>
-    </link>
-    <joint name="top_screen_joint" type="fixed">
-      <parent link="${parent}"/>
-      <child link="top_screen_link"/>
-      <origin xyz="${x} ${y} ${z}" rpy="0 0 0.05"/>
-    </joint>
-  </xacro:macro>
 </robot>

File: src/planning/urdf/main_car/car_radar.xacro (robot description, xacro)
@@ -1,61 +1,29 @@
-<?xml version="1.0"?>
+<!-- 雷达 -->
 <robot xmlns:xacro="http://www.ros.org/wiki/xacro">
-  <xacro:macro name="photo_radar" params="parent x y z radius height">
-    <link name="laser_link">
-      <visual>
-        <origin xyz="0 0 0" rpy="0 0 0"/>
-        <geometry>
-          <cylinder radius="${radius}" length="${height}"/>
-        </geometry>
-        <material name="mat_dark_grey"/>
-      </visual>
-      <visual>
-        <origin xyz="${radius * 0.80} 0 0.005" rpy="0 ${pi / 2.0} 0"/>
-        <geometry>
-          <cylinder radius="0.022" length="0.012"/>
-        </geometry>
-        <material name="mat_black"/>
-      </visual>
-      <visual>
-        <origin xyz="0 0 ${height / 2.0 + 0.004}" rpy="0 0 0"/>
-        <geometry>
-          <cylinder radius="${radius * 0.74}" length="0.008"/>
-        </geometry>
-        <material name="mat_grey"/>
-      </visual>
-      <collision>
-        <origin xyz="0 0 0" rpy="0 0 0"/>
-        <geometry>
-          <cylinder radius="${radius}" length="${height}"/>
-        </geometry>
-      </collision>
-      <xacro:cylinder_inertial_z mass="0.32" radius="${radius}" length="${height}"/>
+    <!-- 雷达尺寸 -->
+    <xacro:property name="radar_radius" value="0.2"/>
+    <xacro:property name="radar_height" value="0.2"/>
+    <!-- 雷达偏移量 -->
+    <xacro:property name="radar_joint_x" value="0.0"/>
+    <xacro:property name="radar_joint_y" value="0.0"/>
+    <xacro:property name="radar_joint_z" value="${car_height / 2.0 + radar_height / 2.0}"/>
+    <!-- 颜色 -->
+    <material name="blue">
+        <color rgba="0.2 0.0 0.7 0.8"/>
+    </material>
+    <!-- 雷达几何 -->
+    <link name="radar">
+        <visual>
+            <geometry>
+                <cylinder radius="${radar_radius}" length="${radar_height}"/>
+            </geometry>
+            <material name="blue"/>
+        </visual>
     </link>
-    <joint name="laser_joint" type="fixed">
-      <parent link="${parent}"/>
-      <child link="laser_link"/>
-      <origin xyz="${x} ${y} ${z}" rpy="0 0 0"/>
+    <!-- 雷达关联到base_link -->
+    <joint name="radar2base_link" type="fixed">
+        <parent link="base_link"/>
+        <child link="radar"/>
+        <origin xyz="${radar_joint_x} ${radar_joint_y} ${radar_joint_z}"/>
     </joint>
-    <link name="rear_lidar_cable_link">
-      <visual>
-        <origin xyz="-0.12 0 0" rpy="0 ${pi / 2.0} 0"/>
-        <geometry>
-          <cylinder radius="0.012" length="0.24"/>
-        </geometry>
-        <material name="mat_dark_grey"/>
-      </visual>
-      <collision>
-        <origin xyz="-0.12 0 0" rpy="0 ${pi / 2.0} 0"/>
-        <geometry>
-          <cylinder radius="0.012" length="0.24"/>
-        </geometry>
-      </collision>
-      <xacro:cylinder_inertial_z mass="0.03" radius="0.012" length="0.24"/>
-    </link>
-    <joint name="rear_lidar_cable_joint" type="fixed">
-      <parent link="laser_link"/>
-      <child link="rear_lidar_cable_link"/>
-      <origin xyz="0 0 0.005" rpy="0 0 0"/>
-    </joint>
-  </xacro:macro>
 </robot>
