Commit message: gazebo colcon

File: src/planning/urdf/main_car/car_base.xacro (robot description, xacro)
@@ -13,7 +13,5 @@
         <color rgba="0.9 0.6 0.0 0.7"/>
     </material>
-    <!-- 根坐标 -->
-    <link name="map"/>
-    <!-- 底盘在map的投影点 -->
+    <!-- 底盘在地面的投影点 (TF 根节点) -->
     <link name="base_footprint"/>
     <!-- 底盘 -->
@@ -26,9 +24,4 @@
         </visual>
     </link>
-    <!-- 投影点关联到地图 -->
-    <joint name="footprint_to_map" type="fixed">
-        <parent link="map"/>
-        <child link="base_footprint"/>
-    </joint>
     <!-- 底盘关联到投影点 -->
     <joint name="base_to_footprint" type="fixed">
